Commit message: fixed urdf of toes

File: src/cerberus_description/urdf/cerberus_final.urdf (robot description, URDF)
Before this commit: robot cerberus, 28 links, 27 joints
Links:
- link lb_toe_link: geometry collision sphere radius=0.012; visual mesh filename=package://cerberus_description/urdf/meshes/toe_own_lb.stl scale=0.001 0.001 0.001
- link lf_toe_link: geometry collision sphere radius=0.012; visual mesh filename=package://cerberus_description/urdf/meshes/toe_own_lf.stl scale=0.001 0.001 0.001
- link rb_toe_link: geometry collision sphere radius=0.012; visual mesh filename=package://cerberus_description/urdf/meshes/toe_own_rb.stl scale=0.001 0.001 0.001
- link rf_toe_link: geometry collision sphere radius=0.012; visual mesh filename=package://cerberus_description/urdf/meshes/toe_own_rf.stl scale=0.001 0.001 0.001
